File: giraffe/honda/nidec_flipped/giraffe20_flipped.sch (EAGLE design)
At the start: 6 parts, among them J3 OBDII-FEMALE-CUT, J4 VERT_RJ45, SW1 4XDPSTSMT

Commit message: Update flipped board
Changed lines of the file:
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@@
 <?xml version="1.0" encoding="utf-8"?>
 <!DOCTYPE eagle SYSTEM "eagle.dtd">
-<eagle version="8.3.2">
+<eagle version="9.2.1">
 <drawing>
 <settings>
@@
 </plain>
 <instances>
-<instance part="J1" gate="G$1" x="63.5" y="101.6"/>
-<instance part="J3" gate="G$1" x="81.28" y="127"/>
-<instance part="J2" gate="G$1" x="157.48" y="101.6"/>
-<instance part="J4" gate="G$1" x="96.52" y="43.18"/>
-<instance part="SW1" gate="G$1" x="175.26" y="134.62"/>
-<instance part="FRAME1" gate="G$1" x="0" y="0"/>
-<instance part="FRAME1" gate="V" x="147.32" y="0"/>
+<instance part="J1" gate="G$1" x="63.5" y="101.6" smashed="yes">
+<attribute name="NAME" x="63.5" y="102.87" size="1.778" layer="95"/>
+</instance>
+<instance part="J3" gate="G$1" x="81.28" y="127" smashed="yes">
+<attribute name="NAME" x="63.754" y="141.224" size="1.778" layer="95"/>
+</instance>
+<instance part="J2" gate="G$1" x="157.48" y="101.6" smashed="yes">
+<attribute name="NAME" x="157.48" y="102.87" size="1.778" layer="95"/>
+</instance>
+<instance part="J4" gate="G$1" x="96.52" y="43.18" smashed="yes">
+<attribute name="NAME" x="100.33" y="53.848" size="1.778" layer="95"/>
+<attribute name="VALUE" x="100.33" y="32.258" size="1.778" layer="96"/>
+</instance>
+<instance part="SW1" gate="G$1" x="175.26" y="134.62" smashed="yes">
+<attribute name="NAME" x="162.56" y="152.4" size="1.9304" layer="95"/>
+</instance>
+<instance part="FRAME1" gate="G$1" x="0" y="0" smashed="yes"/>
+<instance part="FRAME1" gate="V" x="147.32" y="0" smashed="yes">
+<attribute name="LAST_DATE_TIME" x="160.02" y="1.27" size="2.54" layer="94" font="vector"/>
+<attribute name="SHEET" x="233.68" y="1.27" size="2.54" layer="94" font="vector"/>
+<attribute name="DRAWING_NAME" x="162.814" y="17.78" size="2.7432" layer="94" font="vector"/>
+</instance>
 </instances>
 <busses>
@@
 </sheet>
 </sheets>
-<errors>
-</errors>
 </schematic>
 </drawing>
